File: Encoder.kicad_sch (KiCad schematic)
At the start: 2 parts

Commit message: Layed out PCB
Parts:
- C12: footprint (none) -> Capacitor_SMD:C_0402_1005Metric
Changed lines of the file:
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@@
 			)
 		)
-		(property "Footprint" ""
+		(property "Footprint" "Capacitor_SMD:C_0402_1005Metric"
 			(at 125.4252 67.31 0)
 			(effects
